File: hardware/eagle/ublox-lea6-test.brd (EAGLE design)
At the start: 49.5 x 49.5 mm, 52 parts, among them U1 UBLOX-LEA-6T, U2 TPS73633, U3 TPS73633, X1 SERIAL, X2 ANT, X3 FOUT, X4 ANT, X5 FOUT, X6 1PPS, X7 PC, X8 1PPS, X9 22-23-2021

Commit message: Fixed up values and polygon signal
Parts:
- R13: value (none) -> 220R
Routing:
- removed copper zone on layer 1, net N$9
Changed lines of the file:
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@@
 <?xml version="1.0" encoding="utf-8"?>
 <!DOCTYPE eagle SYSTEM "eagle.dtd">
-<eagle version="6.0">
+<eagle version="7.1.0">
 <drawing>
 <settings>
@@
 </class>
 </classes>
-<designrules>
+<designrules name="SeeedStudio_2layer_DRU_no_angle_20140221">
 <description language="de">&lt;b&gt;EAGLE Design Rules&lt;/b&gt;
 &lt;p&gt;
@@
 </description>
 <param name="layerSetup" value="(1*16)"/>
-<param name="mtCopper" value="0.035mm 0.035mm 0.035mm 0.035mm 0.035mm 0.035mm 0.035mm 0.035mm 0.035mm 0.035mm 0.035mm 0.035mm 0.035mm 0.035mm 0.035mm 0.035mm"/>
-<param name="mtIsolate" value="1.5mm 0.15mm 0.2mm 0.15mm 0.2mm 0.15mm 0.2mm 0.15mm 0.2mm 0.15mm 0.2mm 0.15mm 0.2mm 0.15mm 0.2mm"/>
+<param name="mtCopper" value="0.035mm 0.0175mm 0.035mm 0.035mm 0.035mm 0.035mm 0.035mm 0.035mm 0.035mm 0.035mm 0.035mm 0.035mm 0.035mm 0.035mm 0.0175mm 0.035mm"/>
+<param name="mtIsolate" value="1.5mm 1.1mm 0.2mm 0.15mm 0.2mm 0.15mm 0.2mm 0.15mm 0.2mm 0.15mm 0.2mm 0.15mm 0.2mm 0.15mm 0.2mm"/>
 <param name="mdWireWire" value="6mil"/>
 <param name="mdWirePad" value="6mil"/>
@@
 <pass name="Default">
 <param name="RoutingGrid" value="50mil"/>
+<param name="AutoGrid" value="1"/>
+<param name="Efforts" value="0"/>
+<param name="TopRouterVariant" value="1"/>
 <param name="tpViaShape" value="round"/>
 <param name="PrefDir.1" value="|"/>
@@
 </element>
 <element name="LED1" library="led" package="SML0603" value="" x="27.305" y="16.1925"/>
-<element name="R13" library="we_passive" package="0603" value="" x="24.13" y="16.1925"/>
+<element name="R13" library="we_passive" package="0603" value="220R" x="24.13" y="16.1925"/>
 <element name="TP8" library="we_conn" package="TP_1X1" value="TESTPAD" x="8.255" y="34.925" smashed="yes">
 <attribute name="NAME" x="3.8975" y="37.445" size="1.27" layer="25"/>
@@
 <via x="21.9075" y="16.1925" extent="1-16" drill="0.4064"/>
 <wire x1="23.33" y1="16.1925" x2="21.9075" y2="16.1925" width="0.4572" layer="1"/>
+<polygon width="0.3048" layer="1">
+<vertex x="16.8275" y="9.8425"/>
+<vertex x="19.05" y="9.8425"/>
+<vertex x="19.05" y="5.715"/>
+<vertex x="16.51" y="5.715"/>
+<vertex x="16.51" y="9.8425"/>
+</polygon>
 </signal>
 <signal name="1PPS">
@@
 <wire x1="5.23875" y1="30.87" x2="5.23875" y2="31.2675" width="0.6096" layer="1"/>
 </signal>
-<signal name="N$9">
-<polygon width="0.3048" layer="1">
-<vertex x="16.8275" y="9.8425"/>
-<vertex x="19.05" y="9.8425"/>
-<vertex x="19.05" y="5.715"/>
-<vertex x="16.51" y="5.715"/>
-<vertex x="16.51" y="9.8425"/>
-</polygon>
-</signal>
 <signal name="N$27">
